Commit message: urdf with gripper

File: src/igus_rebel_ros2/src/igus_rebel_description/urdf/igus_rebel2.urdf (robot description, URDF)
Before this commit: robot igus_rebel, 12 links, 11 joints
Links:
- added link gripper_base, mass 1.2658; collision cylinder length=0.05 radius=0.04; visual mesh filename=package://igus_rebel_description/meshes/robolink_rebel2/Ele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 scale=0.001 0.001 0.001
- added link gripper_bruecke, mass 1.2658; collision cylinder length=0.05 radius=0.04; visual mesh filename=package://igus_rebel_description/meshes/robolink_rebel2/Bru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 scale=0.001 0.001 0.001
- added link gripper_left, mass 1.2658; collision cylinder length=0.05 radius=0.04; visual mesh filename=package://igus_rebel_description/meshes/robolink_rebel2/Gre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 scale=0.001 0.001 0.001
- added link gripper_right, mass 1.2658; collision cylinder length=0.05 radius=0.04; visual mesh filename=package://igus_rebel_description/meshes/robolink_rebel2/Gre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 scale=0.001 0.001 0.001
- link base_link: geometry collision cylinder length=0.1 radius=0.09; visual mesh filename=package://igus_rebel_description/meshes/robolink_rebel2/bas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
- link link1: geometry collision box size=0.1 0.03 0.1; visual mesh filename=package://igus_rebel_description/meshes/robolink_rebel2/lin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
- link link2: geometry collision cylinder length=0.18 radius=0.06; visual mesh filename=package://igus_rebel_description/meshes/robolink_rebel2/lin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
- link link3: geometry collision box size=0.1 0.03 0.1; visual mesh filename=package://igus_rebel_description/meshes/robolink_rebel2/lin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
- link link4: geometry collision cylinder length=0.1 radius=0.05; visual mesh filename=package://igus_rebel_description/meshes/robolink_rebel2/lin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
- link link5: geometry collision box size=0.1 0.03 0.1; visual mesh filename=package://igus_rebel_description/meshes/robolink_rebel2/lin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
- link link6: geometry collision cylinder length=0.065 radius=0.04; visual mesh filename=package://igus_rebel_description/meshes/robolink_rebel2/lin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
- link motor1: geometry collision cylinder length=0.065 radius=0.05; visual mesh filename=package://igus_rebel_description/meshes/robolink_rebel2/mot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
- link motor2: geometry collision cylinder length=0.065 radius=0.05; visual mesh filename=package://igus_rebel_description/meshes/robolink_rebel2/mot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
- link motor3: geometry collision cylinder length=0.065 radius=0.05; visual mesh filename=package://igus_rebel_description/meshes/robolink_rebel2/mot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
- link motor4: geometry collision cylinder length=0.065 radius=0.05; visual mesh filename=package://igus_rebel_description/meshes/robolink_rebel2/mot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
- link motor5: geometry collision cylinder length=0.065 radius=0.04; visual mesh filename=package://igus_rebel_description/meshes/robolink_rebel2/mot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
Joints:
- added joint gripper_base_joint: type revolute, parent link6, child gripper_base, origin xyz=0 0 0.0515 rpy=0 0 0, axis 0 0 1, limit lower=-3.12414 upper=3.12414 effort=330 velocity=2.16
- added joint gripper_bruecke_joint: type revolute, parent gripper_base, child gripper_bruecke, origin xyz=-0.0225 -0.0425 0.066 rpy=0 0 0, axis 0 0 1, limit lower=-3.12414 upper=3.12414 effort=330 velocity=2.16
- added joint gripper_left_joint: type revolute, parent gripper_bruecke, child gripper_left, origin xyz=0.052 -0.01 -0.0155 rpy=0 -1.57 0, axis 0 0 1, limit lower=-3.12414 upper=3.12414 effort=330 velocity=2.16
- added joint gripper_right_joint: type revolute, parent gripper_bruecke, child gripper_right, origin xyz=-0.011 0.095 -0.0155 rpy=-3.14 -1.57 0, axis 0 0 1, limit lower=-3.12414 upper=3.12414 effort=330 velocity=2.16

Commit message: adjusted urdf

File: src/igus_rebel_ros2/src/igus_rebel_description/urdf/igus_rebel2.urdf (robot description, URDF)
Before this commit: robot igus_rebel, 16 links, 15 joints
Links:
- link gripper_bruecke: geometry visual mesh filename=package://igus_rebel_description/meshes/robolink_rebel2/Bru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 scale=0.001 0.001 0.001
- link gripper_left: geometry collision box size=0.05 0.01 0.05; visual mesh filename=package://igus_rebel_description/meshes/robolink_rebel2/Gre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 scale=0.001 0.001 0.001
- link gripper_right: geometry collision box size=0.05 0.01 0.05; visual mesh filename=package://igus_rebel_description/meshes/robolink_rebel2/Gre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 scale=0.001 0.001 0.001
Joints:
- joint gripper_base_joint: type revolute -> fixed
- joint joint5: type continuous -> revolute

Commit message: gripper urdf and collision

File: src/igus_rebel_ros2/src/igus_rebel_description/urdf/igus_rebel2.urdf (robot description, URDF)
Before this commit: robot igus_rebel, 16 links, 15 joints
Links:
- removed link gripper_bruecke
- link gripper_base: mass 1.2658 -> 0.500; geometry collision box size=0.1 0.13 0.08; visual mesh filename=package://igus_rebel_description/meshes/robolink_rebel2/Gre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 scale=0.001 0.001 0.001
- link gripper_left: mass 1.2658 -> 0.050; geometry collision box size=0.04 0.01 0.043
- link gripper_right: mass 1.2658 -> 0.050; geometry collision box size=0.04 0.01 0.043
Joints:
- removed joint gripper_base_joint
- removed joint gripper_bruecke_joint
- removed joint gripper_left_joint
- removed joint gripper_right_joint
- added joint greifer_fixed_joint: type fixed, parent link6, child gripper_base, origin xyz=0 0 0.12 rpy=0 0 0, axis 0 0 1, limit lower=-3.12414 upper=3.12414 effort=330 velocity=2.16
- added joint gripper_l_joint: type linear, parent gripper_base, child gripper_left, origin xyz=0 0.02 0.04 rpy=0 0 0, axis 0 0 1, limit lower=-3.12414 upper=3.12414 effort=330 velocity=2.16
- added joint gripper_r_joint: type linear, parent gripper_base, child gripper_right, origin xyz=0 -0.02 0.04 rpy=0 0 0, axis 0 0 1, limit lower=-3.12414 upper=3.12414 effort=330 velocity=2.16
